File: Monolith.kicad_sch (KiCad schematic)
At the start: 20 parts, among them J2 Conn_01x11, J3 Conn_01x11, J4 Conn_01x02, J5 Conn_01x02, J6 Conn_01x07, U1 ADS1299IPAGR, U12 ESP32-S3-MINI-1

Commit message: Edit schematic
Parts:
- added C3: 1uF, symbol Device:C
- added R6: 10k, symbol Device:R
Connections:
- net +3V3: now also R6.1
- net EN: now also C3.1, R6.2
- net GND: now also C3.2
Changed lines of the file:
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@@
   (junction (at 213.995 31.75) (diameter 0) (color 0 0 0 0)
+  )
+  (junction (at 168.3004 31.8516) (diameter 0) (color 0 0 0 0)
   )
   (junction (at 82.55 50.165) (diameter 0) (color 0 0 0 0)
@@
     (stroke (width 0) (type default))
   )
+  (wire (pts (xy 168.2496 35.4076) (xy 168.3004 31.8516))
+    (stroke (width 0) (type default))
+  )
+  (wire (pts (xy 168.3004 31.8516) (xy 168.2496 29.3624))
+    (stroke (width 0) (type default))
+  )
   (wire (pts (xy 142.24 146.05) (xy 142.24 143.51))
     (stroke (width 0) (type default))
@@
     (stroke (width 0) (type default))
   )
+  (wire (pts (xy 165.5572 35.4076) (xy 168.2496 35.4076))
+    (stroke (width 0) (type default))
+  )
   (wire (pts (xy 74.93 50.165) (xy 74.93 55.245))
     (stroke (width 0) (type default))
@@
     (stroke (width 0) (type default))
   )
+  (wire (pts (xy 171.6532 31.8516) (xy 168.3004 31.8516))
+    (stroke (width 0) (type default))
+  )
+  (wire (pts (xy 168.2496 29.3624) (xy 165.3032 29.3624))
+    (stroke (width 0) (type default))
+  )
   (wire (pts (xy 151.13 156.21) (xy 144.78 156.21))
     (stroke (width 0) (type default))
@@
     (effects (font (size 1.27 1.27)) (justify right bottom))
   )
+  (label "EN" (at 168.275 53.34 180) (fields_autoplaced)
+    (effects (font (size 1.27 1.27)) (justify right bottom))
+  )
   (label "AVSS" (at 23.495 62.23 180) (fields_autoplaced)
     (effects (font (size 1.27 1.27)) (justify right bottom))
@@
     (effects (font (size 1.27 1.27)) (justify left bottom))
   )
+  (label "EN" (at 171.6532 31.8516 0) (fields_autoplaced)
+    (effects (font (size 1.27 1.27)) (justify left bottom))
+  )
   (label "8N" (at 26.67 111.125 180) (fields_autoplaced)
     (effects (font (size 1.27 1.27)) (justify right bottom))
@@
   (label "5P" (at 46.355 39.37 0) (fields_autoplaced)
     (effects (font (size 1.27 1.27)) (justify left bottom))
-  )
-  (label "EN" (at 168.275 53.34 180) (fields_autoplaced)
-    (effects (font (size 1.27 1.27)) (justify right bottom))
   )
   (label "SRB2" (at 46.355 49.53 0) (fields_autoplaced)
@@
     )
   )
+  (symbol (lib_id "Device:C") (at 165.5572 39.2176 0) (unit 1)
+    (in_bom yes) (on_board yes) (dnp no) (fields_autoplaced)
+    (property "Reference" "C3" (at 168.7322 37.9476 0)
+      (effects (font (size 1.27 1.27)) (justify left))
+    )
+    (property "Value" "1uF" (at 168.7322 40.4876 0)
+      (effects (font (size 1.27 1.27)) (justify left))
+    )
+    (property "Footprint" "" (at 166.5224 43.0276 0)
+      (effects (font (size 1.27 1.27)) hide)
+    )
+    (property "Datasheet" "~" (at 165.5572 39.2176 0)
+      (effects (font (size 1.27 1.27)) hide)
+    )
+    (property "LCSC" "C15849" (at 165.5572 39.2176 0)
+      (effects (font (size 1.27 1.27)) hide)
+    )
+    (pin "1")
+    (pin "2")
+    (instances
+      (project "Monolith"
+        (path "/a4ecfbe3-0f16-403e-8cdc-2760bb3b2c3f"
+          (reference "C3") (unit 1)
+        )
+      )
+    )
+  )
   (symbol (lib_id "power:+3V3") (at 143.764 29.21 270) (unit 1)
     (in_bom yes) (on_board yes) (dnp no) (fields_autoplaced)
@@
     )
   )
+  (symbol (lib_id "power:+3V3") (at 165.3032 21.7424 0) (unit 1)
+    (in_bom yes) (on_board yes) (dnp no) (fields_autoplaced)
+    (property "Reference" "#PWR014" (at 165.3032 25.5524 0)
+      (effects (font (size 1.27 1.27)) hide)
+    )
+    (property "Value" "+3V3" (at 165.3032 16.6624 0)
+      (effects (font (size 1.27 1.27)))
+    )
+    (property "Footprint" "" (at 165.3032 21.7424 0)
+      (effects (font (size 1.27 1.27)) hide)
+    )
+    (property "Datasheet" "" (at 165.3032 21.7424 0)
+      (effects (font (size 1.27 1.27)) hide)
+    )
+    (pin "1")
+    (instances
+      (project "Monolith"
+        (path "/a4ecfbe3-0f16-403e-8cdc-2760bb3b2c3f"
+          (reference "#PWR014") (unit 1)
+        )
+      )
+    )
+  )
+  (symbol (lib_id "power:GND") (at 165.5572 43.0276 0) (unit 1)
+    (in_bom yes) (on_board yes) (dnp no) (fields_autoplaced)
+    (property "Reference" "#PWR013" (at 165.5572 49.3776 0)
+      (effects (font (size 1.27 1.27)) hide)
+    )
+    (property "Value" "GND" (at 165.5572 47.5488 0)
+      (effects (font (size 1.27 1.27)))
+    )
+    (property "Footprint" "" (at 165.5572 43.0276 0)
+      (effects (font (size 1.27 1.27)) hide)
+    )
+    (property "Datasheet" "" (at 165.5572 43.0276 0)
+      (effects (font (size 1.27 1.27)) hide)
+    )
+    (pin "1")
+    (instances
+      (project "Monolith"
+        (path "/a4ecfbe3-0f16-403e-8cdc-2760bb3b2c3f"
+          (reference "#PWR013") (unit 1)
+        )
+      )
+    )
+  )
   (symbol (lib_id "Device:C") (at 155.575 138.43 270) (unit 1)
     (in_bom yes) (on_board yes) (dnp no) (fields_autoplaced)
@@
         )
       )
+    )
+  )
+  (symbol (lib_id "Device:R") (at 165.3032 25.5524 0) (unit 1)
+    (in_bom yes) (on_board yes) (dnp no) (fields_autoplaced)
+    (property "Reference" "R6" (at 167.2336 24.2824 0)
+      (effects (font (size 1.27 1.27)) (justify left))
+    )
+    (property "Value" "10k" (at 167.2336 26.8224 0)
+      (effects (font (size 1.27 1.27)) (justify left))
+    )
+    (property "Footprint" "" (at 163.5252 25.5524 90)
+      (effects (font (size 1.27 1.27)) hide)
+    )
+    (property "Datasheet" "~" (at 165.3032 25.5524 0)
+      (effects (font (size 1.27 1.27)) hide)
+    )
+    (property "LCSC" "C98220" (at 165.3032 25.5524 0)
+      (effects (font (size 1.27 1.27)) hide)
+    )
+    (pin "1")
+    (pin "2")
+    (instances
+      (project "Monolith"
+        (path "/a4ecfbe3-0f16-403e-8cdc-2760bb3b2c3f"
+          (reference "R6") (unit 1)
+        )
+      )
