File: ADSPower.kicad_sch (KiCad schematic)
At the start: 20 parts, among them U4 LM2664M6, U6 TLV70025QDDCRQ1, U7 TPS72325

Commit message: fix pick and place stuff
Parts:
- C19, C40, C42, C44, C47: LCSC C172735 -> C3011705
- C39, C41, C43, C48: LCSC C5189821 -> C15849
Changed lines of the file:
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@@
       (effects (font (size 1.27 1.27)) hide)
     )
-    (property "LCSC" "C172735" (at 87.63 107.95 0)
+    (property "LCSC" "C3011705" (at 87.63 107.95 0)
       (effects (font (size 1.27 1.27)) hide)
     )
@@
       (effects (font (size 1.27 1.27)) hide)
     )
-    (property "LCSC" "C172735" (at 182.88 76.2 0)
+    (property "LCSC" "C3011705" (at 182.88 76.2 0)
       (effects (font (size 1.27 1.27)) hide)
     )
@@
       (effects (font (size 1.27 1.27)) hide)
     )
-    (property "LCSC" "C172735" (at 62.23 107.95 0)
+    (property "LCSC" "C3011705" (at 62.23 107.95 0)
       (effects (font (size 1.27 1.27)) hide)
     )
@@
       (effects (font (size 1.27 1.27)) hide)
     )
-    (property "LCSC" "C5189821" (at 76.835 107.95 0)
+    (property "LCSC" "C15849" (at 76.835 107.95 0)
       (effects (font (size 1.27 1.27)) hide)
     )
@@
       (effects (font (size 1.27 1.27)) hide)
     )
-    (property "LCSC" "C172735" (at 86.995 129.54 0)
+    (property "LCSC" "C3011705" (at 86.995 129.54 0)
       (effects (font (size 1.27 1.27)) hide)
     )
@@
       (effects (font (size 1.27 1.27)) hide)
     )
-    (property "LCSC" "C5189821" (at 51.435 107.95 0)
+    (property "LCSC" "C15849" (at 51.435 107.95 0)
       (effects (font (size 1.27 1.27)) hide)
     )
@@
       (effects (font (size 1.27 1.27)) hide)
     )
-    (property "LCSC" "C5189821" (at 76.2 129.54 0)
+    (property "LCSC" "C15849" (at 76.2 129.54 0)
       (effects (font (size 1.27 1.27)) hide)
     )
@@
       (effects (font (size 1.27 1.27)) hide)
     )
-    (property "LCSC" "C5189821" (at 50.8 128.27 0)
+    (property "LCSC" "C15849" (at 50.8 128.27 0)
       (effects (font (size 1.27 1.27)) hide)
     )
@@
       (effects (font (size 1.27 1.27)) hide)
     )
-    (property "LCSC" "C172735" (at 61.595 128.27 0)
-      (effects (font (size 1.27 1.27)) hide)
-    )
+    (property "LCSC" "C3011705" (at 61.595 128.27 0)
+      (effects (font (size 1.27 1.27)) hide)
+    )

Commit message: new fixes
Parts:
- C19, C40, C42, C44, C47: LCSC C3011705 -> C14663
- C20, C28, C29, C33: LCSC C5189827 -> C23630
- C30, C31, C32, C34: LCSC C1691 -> C96446
Changed lines of the file:
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@@
       (effects (font (size 1.27 1.27)) hide)
     )
-    (property "LCSC" "C1691" (at 238.76 110.49 0)
+    (property "LCSC" "C96446" (at 238.76 110.49 0)
       (effects (font (size 1.27 1.27)) hide)
     )
@@
       (effects (font (size 1.27 1.27)) hide)
     )
-    (property "LCSC" "C3011705" (at 87.63 107.95 0)
+    (property "LCSC" "C14663" (at 87.63 107.95 0)
       (effects (font (size 1.27 1.27)) hide)
     )
@@
       (effects (font (size 1.27 1.27)) hide)
     )
-    (property "LCSC" "C5189827" (at 221.615 110.49 0)
+    (property "LCSC" "C23630" (at 221.615 110.49 0)
       (effects (font (size 1.27 1.27)) hide)
     )
@@
       (effects (font (size 1.27 1.27)) hide)
     )
-    (property "LCSC" "C1691" (at 212.725 64.135 0)
+    (property "LCSC" "C96446" (at 212.725 64.135 0)
       (effects (font (size 1.27 1.27)) hide)
     )
@@
       (effects (font (size 1.27 1.27)) hide)
     )
-    (property "LCSC" "C3011705" (at 182.88 76.2 0)
+    (property "LCSC" "C14663" (at 182.88 76.2 0)
       (effects (font (size 1.27 1.27)) hide)
     )
@@
       (effects (font (size 1.27 1.27)) hide)
     )
-    (property "LCSC" "C5189827" (at 139.7 59.69 0)
+    (property "LCSC" "C23630" (at 139.7 59.69 0)
       (effects (font (size 1.27 1.27)) hide)
     )
@@
       (effects (font (size 1.27 1.27)) hide)
     )
-    (property "LCSC" "C3011705" (at 62.23 107.95 0)
+    (property "LCSC" "C14663" (at 62.23 107.95 0)
       (effects (font (size 1.27 1.27)) hide)
     )
@@
       (effects (font (size 1.27 1.27)) hide)
     )
-    (property "LCSC" "C3011705" (at 86.995 129.54 0)
+    (property "LCSC" "C14663" (at 86.995 129.54 0)
       (effects (font (size 1.27 1.27)) hide)
     )
@@
       (effects (font (size 1.27 1.27)) hide)
     )
-    (property "LCSC" "C1691" (at 100.965 67.31 0)
+    (property "LCSC" "C96446" (at 100.965 67.31 0)
       (effects (font (size 1.27 1.27)) hide)
     )
@@
       (effects (font (size 1.27 1.27)) hide)
     )
-    (property "LCSC" "C5189827" (at 197.485 64.135 0)
+    (property "LCSC" "C23630" (at 197.485 64.135 0)
       (effects (font (size 1.27 1.27)) hide)
     )
@@
       (effects (font (size 1.27 1.27)) hide)
     )
-    (property "LCSC" "C1691" (at 48.26 69.85 0)
+    (property "LCSC" "C96446" (at 48.26 69.85 0)
       (effects (font (size 1.27 1.27)) hide)
     )
@@
       (effects (font (size 1.27 1.27)) hide)
     )
-    (property "LCSC" "C5189827" (at 131.445 116.205 0)
+    (property "LCSC" "C23630" (at 131.445 116.205 0)
       (effects (font (size 1.27 1.27)) hide)
     )
@@
       (effects (font (size 1.27 1.27)) hide)
     )
-    (property "LCSC" "C3011705" (at 61.595 128.27 0)
-      (effects (font (size 1.27 1.27)) hide)
-    )
+    (property "LCSC" "C14663" (at 61.595 128.27 0)
+      (effects (font (size 1.27 1.27)) hide)
+    )
