File: ArrayFilter.kicad_sch (KiCad schematic)
At the start: 2 parts

Commit message: new fixes
Parts:
- removed R?: CAT10-222J4LF, CAT10-222J4LF:RESCAV50P200X100X55-8N, symbol CAT10-222J4LF:CAT10-222J4LF
- added R10, R15, R21, R4: R 2.2k, Capacitor_SMD:C_0402_1005Metric, symbol Device:R
Connections:
- net IN1: now also R4.1
- net IN2: now also R10.1
- net IN3: now also R15.1
- net IN4: now also R21.1
- net OUT1: now also R4.2
- net OUT2: now also R10.2
- net OUT3: now also R15.2
- net OUT4: now also R21.2
- net GNDA renamed SRB1
