File: Electrodes.kicad_sch (KiCad schematic)
At the start: 6 parts

Commit message: new fixes
Other:
- sheet ArrayFilter ports: added SRB1; removed none
- sheet ArrayFilter1 ports: added SRB1; removed none
- sheet ArrayFilter2 ports: added SRB1; removed none
- sheet ArrayFilter3 ports: added SRB1; removed none
- sheet ArrayFilter4 ports: added SRB1; removed none
Changed lines of the file:
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@@
   (no_connect (at 23.241 183.515))
   (no_connect (at 23.241 188.595))
+  (wire (pts (xy 78.105 87.63) (xy 78.105 89.789))
+    (stroke (width 0) (type default))
+  )
+  (wire (pts (xy 78.105 123.825) (xy 78.105 126.238))
+    (stroke (width 0) (type default))
+  )
+  (wire (pts (xy 78.105 51.435) (xy 78.105 53.467))
+    (stroke (width 0) (type default))
+  )
+  (wire (pts (xy 78.105 160.655) (xy 78.105 163.195))
+    (stroke (width 0) (type default))
+  )
+  (wire (pts (xy 78.105 15.24) (xy 78.105 17.399))
+    (stroke (width 0) (type default))
+  )
   (hierarchical_label "SRB1" (shape input) (at 65.151 166.624 180) (fields_autoplaced)
     (effects (font (size 1.27 1.27)) (justify right))
@@
     (effects (font (size 1.27 1.27)) (justify left))
   )
+  (hierarchical_label "INSRB1" (shape input) (at 78.105 160.655 0) (fields_autoplaced)
+    (effects (font (size 1.27 1.27)) (justify left))
+  )
   (hierarchical_label "1P" (shape input) (at 23.241 20.955 180) (fields_autoplaced)
     (effects (font (size 1.27 1.27)) (justify right))
@@
     (effects (font (size 1.27 1.27)) (justify left))
   )
+  (hierarchical_label "INSRB1" (shape input) (at 78.105 87.63 0) (fields_autoplaced)
+    (effects (font (size 1.27 1.27)) (justify left))
+  )
   (hierarchical_label "6N" (shape input) (at 65.405 116.205 180) (fields_autoplaced)
     (effects (font (size 1.27 1.27)) (justify right))
@@
     (effects (font (size 1.27 1.27)) (justify right))
   )
+  (hierarchical_label "INSRB1" (shape input) (at 78.105 15.24 0) (fields_autoplaced)
+    (effects (font (size 1.27 1.27)) (justify left))
+  )
   (hierarchical_label "3P" (shape input) (at 65.659 56.896 180) (fields_autoplaced)
     (effects (font (size 1.27 1.27)) (justify right))
@@
   (hierarchical_label "5P" (shape input) (at 65.405 93.218 180) (fields_autoplaced)
     (effects (font (size 1.27 1.27)) (justify right))
+  )
+  (hierarchical_label "INSRB1" (shape input) (at 78.105 123.825 0) (fields_autoplaced)
+    (effects (font (size 1.27 1.27)) (justify left))
+  )
+  (hierarchical_label "INSRB1" (shape input) (at 78.105 51.435 0) (fields_autoplaced)
+    (effects (font (size 1.27 1.27)) (justify left))
   )
   (hierarchical_label "5P" (shape input) (at 23.241 86.995 180) (fields_autoplaced)
@@
       (effects (font (size 1.27 1.27)) (justify left))
     )
+    (pin "SRB1" input (at 78.105 89.789 90)
+      (effects (font (size 1.27 1.27)) (justify right))
+    )
     (instances
       (project "Monolith"
@@
       (effects (font (size 1.27 1.27)) (justify left))
     )
+    (pin "SRB1" input (at 78.105 53.467 90)
+      (effects (font (size 1.27 1.27)) (justify right))
+    )
     (instances
       (project "Monolith"
@@
       (effects (font (size 1.27 1.27)) (justify left))
     )
+    (pin "SRB1" input (at 78.105 163.195 90)
+      (effects (font (size 1.27 1.27)) (justify right))
+    )
     (instances
       (project "Monolith"
@@
       (effects (font (size 1.27 1.27)) (justify left))
     )
+    (pin "SRB1" input (at 78.105 17.399 90)
+      (effects (font (size 1.27 1.27)) (justify right))
+    )
     (instances
       (project "Monolith"
@@
       (effects (font (size 1.27 1.27)) (justify left))
     )
-    (instances
+    (pin "SRB1" input (at 78.105 126.238 90)
+      (effects (font (size 1.27 1.27)) (justify right))
+    )
+    (instances
