File: USBPort.kicad_sch (KiCad schematic)
At the start: 12 parts, among them IC1 HT7550-1, J1 USB_B_Micro

Commit message: fix pick and place stuff
Parts:
- C22, C23: LCSC C172735 -> C3011705
Changed lines of the file:
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@@
       (effects (font (size 1.27 1.27)) hide)
     )
-    (property "LCSC" "C172735" (at 132.715 75.565 0)
+    (property "LCSC" "C3011705" (at 132.715 75.565 0)
       (effects (font (size 1.27 1.27)) hide)
     )
@@
       (effects (font (size 1.27 1.27)) hide)
     )
-    (property "LCSC" "C172735" (at 132.715 60.325 0)
+    (property "LCSC" "C3011705" (at 132.715 60.325 0)
       (effects (font (size 1.27 1.27)) hide)
     )

Commit message: fix usb
Parts:
- J1: footprint Connector_USB:USB_Micro-B_Amphenol_10103594-0001LF_Horizontal -> Connector_USB:USB_Micro-B_Amphenol_10118194_Horizontal; LCSC C428495 -> C132563
Changed lines of the file:
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@@
       (effects (font (size 1.27 1.27)) (justify right))
     )
-    (property "Footprint" "Connector_USB:USB_Micro-B_Amphenol_10103594-0001LF_Horizontal" (at 168.275 85.725 0)
+    (property "Footprint" "Connector_USB:USB_Micro-B_Amphenol_10118194_Horizontal" (at 168.275 85.725 0)
       (effects (font (size 1.27 1.27)) hide)
     )
@@
       (effects (font (size 1.27 1.27)) hide)
     )
-    (property "LCSC" "C428495" (at 172.085 84.455 0)
+    (property "LCSC" "C132563" (at 172.085 84.455 0)
       (effects (font (size 1.27 1.27)) hide)
     )

Commit message: Edit schematic
Parts:
- removed IC1: HT7550-1, HT7550-1:SOT89, symbol HT7550-1:HT7550-1
- added U2: AMS1117-3.3, AMS1117-3.3:SOT229P700X180-4N, symbol Regulator_Linear:AMS1117-3.3
Connections:
- net +3V3: now also U2.2 (VO)
- net GND: now also U2.1 (GND)
- net at C21.2, C22.2, D11.C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: now also U2.3 (VI)
Changed lines of the file:
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@@
   (junction (at 150.495 64.135) (diameter 0) (color 0 0 0 0)
   )
+  (junction (at 132.715 56.515) (diameter 0) (color 0 0 0 0)
+  )
   (junction (at 150.495 56.515) (diameter 0) (color 0 0 0 0)
   )
   (junction (at 161.925 79.375) (diameter 0) (color 0 0 0 0)
-  )
-  (junction (at 132.715 56.515) (diameter 0) (color 0 0 0 0)
   )
   (junction (at 160.655 56.515) (diameter 0) (color 0 0 0 0)
@@
     (stroke (width 0) (type default))
   )
-  (wire (pts (xy 118.745 79.375) (xy 118.745 56.515))
+  (wire (pts (xy 115.316 79.375) (xy 115.316 56.515))
     (stroke (width 0) (type default))
   )
@@
     (stroke (width 0) (type default))
   )
-  (wire (pts (xy 123.825 56.515) (xy 132.715 56.515))
+  (wire (pts (xy 122.936 48.895) (xy 124.587 48.895))
+    (stroke (width 0) (type default))
+  )
+  (wire (pts (xy 132.715 41.275) (xy 132.715 56.515))
     (stroke (width 0) (type default))
   )
@@
     (stroke (width 0) (type default))
   )
-  (wire (pts (xy 132.715 79.375) (xy 118.745 79.375))
+  (wire (pts (xy 132.715 79.375) (xy 115.316 79.375))
     (stroke (width 0) (type default))
   )
@@
   )
   (wire (pts (xy 132.715 56.515) (xy 150.495 56.515))
+    (stroke (width 0) (type default))
+  )
+  (wire (pts (xy 115.316 41.275) (xy 132.715 41.275))
     (stroke (width 0) (type default))
   )
@@
   (hierarchical_label "CHIP_PU" (shape input) (at 168.275 136.525 270) (fields_autoplaced)
     (effects (font (size 1.27 1.27)) (justify right))
-  )
-  (symbol (lib_id "HT7550-1:HT7550-1") (at 118.745 51.435 0) (unit 1)
-    (in_bom yes) (on_board yes) (dnp no) (fields_autoplaced)
-    (property "Reference" "IC1" (at 130.175 45.72 0)
-      (effects (font (size 1.27 1.27)) (justify left))
-    )
-    (property "Value" "HT7550-1" (at 130.175 48.26 0)
-      (effects (font (size 1.27 1.27)) (justify left))
-    )
-    (property "Footprint" "HT7550-1:SOT89" (at 118.745 51.435 0)
-      (effects (font (size 1.27 1.27)) (justify bottom) hide)
-    )
-    (property "Datasheet" "" (at 118.745 51.435 0)
-      (effects (font (size 1.27 1.27)) hide)
-    )
-    (property "MF" "Holtek" (at 118.745 51.435 0)
-      (effects (font (size 1.27 1.27)) (justify bottom) hide)
-    )
-    (property "Description" "\nVoltage stabiliser; LDO, fixed; 5V; 0.1A; SOT89; SMD\n" (at 118.745 51.435 0)
-      (effects (font (size 1.27 1.27)) (justify bottom) hide)
-    )
-    (property "Package" "None" (at 118.745 51.435 0)
-      (effects (font (size 1.27 1.27)) (justify bottom) hide)
-    )
-    (property "Price" "None" (at 118.745 51.435 0)
-      (effects (font (size 1.27 1.27)) (justify bottom) hide)
-    )
-    (property "SnapEDA_Link" "https://www.snapeda.com/parts/HT7550-1/Holtek/view-part/?ref=snap" (at 118.745 51.435 0)
-      (effects (font (size 1.27 1.27)) (justify bottom) hide)
-    )
-    (property "MP" "HT7550-1" (at 118.745 51.435 0)
-      (effects (font (size 1.27 1.27)) (justify bottom) hide)
-    )
-    (property "Availability" "Not in stock" (at 118.745 51.435 0)
-      (effects (font (size 1.27 1.27)) (justify bottom) hide)
-    )
-    (property "Check_prices" "https://www.snapeda.com/parts/HT7550-1/Holtek/view-part/?ref=eda" (at 118.745 51.435 0)
-      (effects (font (size 1.27 1.27)) (justify bottom) hide)
-    )
-    (property "LCSC" "C16106" (at 118.745 51.435 0)
-      (effects (font (size 1.27 1.27)) hide)
-    )
-    (pin "1")
-    (pin "2")
-    (pin "2@1")
-    (pin "3")
-    (instances
-      (project "Monolith"
-        (path "/a4ecfbe3-0f16-403e-8cdc-2760bb3b2c3f"
-          (reference "IC1") (unit 1)
-        )
-        (path "/a4ecfbe3-0f16-403e-8cdc-2760bb3b2c3f/14efd714-8e75-4017-9994-542d74377c4f"
-          (reference "IC1") (unit 1)
-        )
-      )
-    )
   )
   (symbol (lib_id "Device:C") (at 132.715 75.565 0) (unit 1)
@@
     )
   )
-  (symbol (lib_id "power:GND") (at 113.665 56.515 0) (unit 1)
-    (in_bom yes) (on_board yes) (dnp no) (fields_autoplaced)
-    (property "Reference" "#PWR028" (at 113.665 62.865 0)
-      (effects (font (size 1.27 1.27)) hide)
-    )
-    (property "Value" "GND" (at 113.665 61.595 0)
-      (effects (font (size 1.27 1.27)))
-    )
-    (property "Footprint" "" (at 113.665 56.515 0)
-      (effects (font (size 1.27 1.27)) hide)
-    )
-    (property "Datasheet" "" (at 113.665 56.515 0)
+  (symbol (lib_id "power:GND") (at 124.587 48.895 90) (unit 1)
+    (in_bom yes) (on_board yes) (dnp no) (fields_autoplaced)
+    (property "Reference" "#PWR028" (at 130.937 48.895 0)
+      (effects (font (size 1.27 1.27)) hide)
+    )
+    (property "Value" "GND" (at 127.762 48.895 90)
+      (effects (font (size 1.27 1.27)) (justify right))
+    )
+    (property "Footprint" "" (at 124.587 48.895 0)
+      (effects (font (size 1.27 1.27)) hide)
+    )
+    (property "Datasheet" "" (at 124.587 48.895 0)
       (effects (font (size 1.27 1.27)) hide)
     )
@@
         )
       )
+    )
+  )
+  (symbol (lib_id "Regulator_Linear:AMS1117-3.3") (at 115.316 48.895 90) (unit 1)
+    (in_bom yes) (on_board yes) (dnp no) (fields_autoplaced)
+    (property "Reference" "U2" (at 112.141 47.625 90)
+      (effects (font (size 1.27 1.27)) (justify left))
+    )
+    (property "Value" "AMS1117-3.3" (at 112.141 50.165 90)
+      (effects (font (size 1.27 1.27)) (justify left))
+    )
+    (property "Footprint" "AMS1117-3.3:SOT229P700X180-4N" (at 110.236 48.895 0)
+      (effects (font (size 1.27 1.27)) hide)
+    )
+    (property "Datasheet" "http://www.advanced-monolithic.com/pdf/ds1117.pdf" (at 121.666 46.355 0)
+      (effects (font (size 1.27 1.27)) hide)
+    )
+    (property "LCSC" "C347222" (at 115.316 48.895 90)
+      (effects (font (size 1.27 1.27)) hide)
+    )
+    (pin "1")
+    (pin "2")
+    (pin "3")
+    (instances
+      (project "Monolith"
+        (path "/a4ecfbe3-0f16-403e-8cdc-2760bb3b2c3f/14efd714-8e75-4017-9994-542d74377c4f"
+          (reference "U2") (unit 1)
+        )
+      )

Commit message: fix led
Parts:
- D7: LCSC C189307 -> C84259
Changed lines of the file:
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@@
       (effects (font (size 1.27 1.27)) hide)
     )
-    (property "LCSC" "C189307" (at 175.895 62.865 90)
+    (property "LCSC" "C84259" (at 175.895 62.865 90)
       (effects (font (size 1.27 1.27)) hide)
     )

Commit message: new fixes
Parts:
- removed D10, D8, D9: LESD5D5.0CT1G, LESD5D5.0CT1G:TVS_LESD5D5.0CT1G, symbol LESD5D5.0CT1G:LESD5D5.0CT1G
- added D?: TPD4E1B06DCKR, TPD4E1B06DCKR:TVS_TPD4E1B06DCKR, symbol TPD4E1B06DCKR:TPD4E1B06DCKR
- C21, C24: LCSC C1691 -> C96446
- C22, C23: LCSC C3011705 -> C14663
- D11: LCSC C82544 -> C8598
- D7: value BLUE LED -> EMERALD LED; LCSC C84259 -> C2297
- R17: value 5.1 -> 100; LCSC C114626 -> C22775
Connections:
- net GND: now also D?.3
- net at C21.2, C22.2, D11.C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: now also D?.4
- net USBtoUART/DN renamed DN
- net DN: now also D?.2
- net USBtoUART/DP renamed DP
- net DP: now also D?.1
- no-connect marks 1 -> 2
Other:
- removed sheet USBtoUART
