File: USBtoUART.kicad_sch (KiCad schematic)
At the start: 12 parts, among them Q1 BC818, Q2 BC818, U3 CP2102N-A02-GQFN28R

Commit message: fix pick and place stuff
Parts:
- C21: LCSC C5189821 -> C15849
- C23: LCSC C172735 -> C3011705
Changed lines of the file:
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@@
       (effects (font (size 1.27 1.27)) hide)
     )
-    (property "LCSC" "C172735" (at 194.31 64.77 0)
+    (property "LCSC" "C3011705" (at 194.31 64.77 0)
       (effects (font (size 1.27 1.27)) hide)
     )
@@
       (effects (font (size 1.27 1.27)) hide)
     )
-    (property "LCSC" "C5189821" (at 100.33 96.52 0)
-      (effects (font (size 1.27 1.27)) hide)
-    )
+    (property "LCSC" "C15849" (at 100.33 96.52 0)
+      (effects (font (size 1.27 1.27)) hide)
+    )

Commit message: new fixes
Parts:
- C22: LCSC C560882 -> C1779
- C23: LCSC C3011705 -> C14663
- Q1, Q2: LCSC C154797 -> C2150
- R17: value R 22.1k (1%) -> R 22k; LCSC C137768 -> C31850
- R22: value R 47.5k (1%) -> R 47k; LCSC C136962 -> C25819
- R23: LCSC C22548 -> C21190
- R24, R25, R26: LCSC C98220 -> C25804
Changed lines of the file:
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@@
       (effects (font (size 1.27 1.27)) hide)
     )
-    (property "LCSC" "C22548" (at 118.11 72.39 90)
+    (property "LCSC" "C21190" (at 118.11 72.39 90)
       (effects (font (size 1.27 1.27)) hide)
     )
@@
       (effects (font (size 1.27 1.27)) (justify left) hide)
     )
-    (property "LCSC" "C154797" (at 228.6 105.41 0)
+    (property "LCSC" "C2150" (at 228.6 105.41 0)
       (effects (font (size 1.27 1.27)) hide)
     )
@@
       (effects (font (size 1.27 1.27)) hide)
     )
-    (property "LCSC" "C98220" (at 214.63 105.41 90)
+    (property "LCSC" "C25804" (at 214.63 105.41 90)
       (effects (font (size 1.27 1.27)) hide)
     )
@@
       (effects (font (size 1.27 1.27)) hide)
     )
-    (property "LCSC" "C98220" (at 214.63 87.63 90)
+    (property "LCSC" "C25804" (at 214.63 87.63 90)
       (effects (font (size 1.27 1.27)) hide)
     )
@@
       (effects (font (size 1.27 1.27)) hide)
     )
-    (property "LCSC" "C98220" (at 191.77 76.2 90)
+    (property "LCSC" "C25804" (at 191.77 76.2 90)
       (effects (font (size 1.27 1.27)) hide)
     )
@@
       (effects (font (size 1.27 1.27)) hide)
     )
-    (property "LCSC" "C3011705" (at 194.31 64.77 0)
+    (property "LCSC" "C14663" (at 194.31 64.77 0)
       (effects (font (size 1.27 1.27)) hide)
     )
@@
       (effects (font (size 1.27 1.27)))
     )
-    (property "Value" "R 22.1k (1%)" (at 71.12 87.63 90)
+    (property "Value" "R 22k" (at 71.12 87.63 90)
       (effects (font (size 1.27 1.27)))
     )
@@
       (effects (font (size 1.27 1.27)) hide)
     )
-    (property "LCSC" "C137768" (at 71.12 90.17 90)
+    (property "LCSC" "C31850" (at 71.12 90.17 90)
       (effects (font (size 1.27 1.27)) hide)
     )
@@
       (effects (font (size 1.27 1.27)) (justify left))
     )
-    (property "Value" "R 47.5k (1%)" (at 82.55 98.425 0)
+    (property "Value" "R 47k" (at 82.55 98.425 0)
       (effects (font (size 1.27 1.27)) (justify left))
     )
@@
       (effects (font (size 1.27 1.27)) hide)
     )
-    (property "LCSC" "C136962" (at 80.01 96.52 0)
+    (property "LCSC" "C25819" (at 80.01 96.52 0)
       (effects (font (size 1.27 1.27)) hide)
     )
@@
       (effects (font (size 1.27 1.27)) hide)
     )
-    (property "LCSC" "C560882" (at 182.88 64.77 0)
+    (property "LCSC" "C1779" (at 182.88 64.77 0)
       (effects (font (size 1.27 1.27)) hide)
     )
@@
       (effects (font (size 1.27 1.27)) (justify left) hide)
     )
-    (property "LCSC" "C154797" (at 228.6 87.63 0)
-      (effects (font (size 1.27 1.27)) hide)
-    )
+    (property "LCSC" "C2150" (at 228.6 87.63 0)
+      (effects (font (size 1.27 1.27)) hide)
+    )
