File: Monolith.kicad_pcb (KiCad board)
At the start: 2 copper layers, 89.9 x 42.7 mm, 82 parts, among them J1 USB_B_Micro, J2 Conn_01x11, J3 Conn_01x11, J4 Conn_01x02, J5 Conn_01x02, J7 Conn_01x08, Q1 BC818, Q2 BC818, U1 ADS1299IPAGR, U12 ESP32-S3-MINI-1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

Commit message: fixes
Parts:
- C20: value 1uF -> 0.1uF
- moved C40 1.45 mm to (227.7, 150.4)
- moved C41 1.45 mm to (226.7, 158.6)
- moved C42 1.45 mm to (227.7, 152.5)
- moved C43 1.45 mm to (223.9, 152.5)
- moved C44 1.45 mm to (223.4, 158.6)
- moved C45 1.45 mm to (229.7, 160.0)
- moved C46 1.45 mm to (229.7, 156.9)
- moved C47 1.45 mm to (223.9, 151.0)
- moved C49 1.45 mm to (237.8, 156.5)
- moved C55 1.45 mm to (240.9, 151.0)
- moved U4 1.45 mm to (232.9, 158.0)
- moved C39 1.45 mm to (226.7, 156.1)
- moved C48 1.45 mm to (223.4, 156.0)
- moved C50 1.45 mm to (232.4, 154.6)
- moved C51 1.45 mm to (230.4, 151.6)
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Connections:
- C32 pad 1: Net-(U1-VREFN) -> /AVSS
- C33 pad 1: Net-(U1-VREFN) -> /AVSS
- U1 pad 25: Net-(U1-VREFN) -> /AVSS
Routing:
- net +3V3: track 222.7 -> 185.7 mm, vias 15 -> 14
- net Net-(U1-VREFN): track 12.0 -> 0.00 mm, vias 2 -> 0
- net /AVDD: track 109.6 -> 105.1 mm, vias 6 -> 7
- net /AVSS: track 108.6 -> 112.9 mm, vias 0 -> 2
- net Net-(U1-VREFP): track 9.80 -> 8.70 mm
- net Net-(U1-VCAP4): track 7.92 -> 7.15 mm, vias 2 -> 0
- net GNDA: track 195.4 -> 194.8 mm
- net Net-(U1-VCAP3): track 22.7 -> 22.2 mm
- net Net-(U1-VCAP2): track 6.32 -> 5.79 mm
- net Net-(U1-VCAP1): track 5.69 -> 5.15 mm, vias 0 -> 2

Commit message: fixes
Parts:
- moved D7 0.52 mm to (207.9, 144.8)
Routing:
- net +3V3: track 185.7 -> 212.5 mm, vias 14 -> 15
Changed lines of the file:
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@@
   )
   (footprint "LESD5D5.0CT1G:TVS_LESD5D5.0CT1G" (layer "F.Cu")
-    (at 207.862706 144.257929 180)
+    (at 207.862706 144.78 180)
     (property "Availability" "Not in stock")
     (property "Check_prices" "https://www.snapeda.com/parts/LESD5D5.0CT1G/Leshan+Radio+Co./view-part/?ref=eda")
@@
   (segment (start 230.632 147.775) (end 230.632 148.7685) (width 0.25) (layer "F.Cu") (net 32))
   (segment (start 229.414 145.638) (end 229.414 144.764941) (width 0.25) (layer "F.Cu") (net 32))
+  (segment (start 234.188 160.528) (end 234.188 159.030998) (width 0.25) (layer "F.Cu") (net 32))
   (segment (start 199.6014 130.7932) (end 199.6014 129.956674) (width 0.25) (layer "F.Cu") (net 32))
   (segment (start 230.414 145.638) (end 230.414 147.557) (width 0.25) (layer "F.Cu") (net 32))
@@
   (segment (start 206.533217 136.500256) (end 205.509296 135.476335) (width 0.25) (layer "F.Cu") (net 32))
   (segment (start 201.220838 131.614665) (end 202.183457 130.652046) (width 0.25) (layer "F.Cu") (net 32))
+  (segment (start 234.188 159.030998) (end 234.28 158.938998) (width 0.25) (layer "F.Cu") (net 32))
   (segment (start 238.168999 156.982001) (end 237.836 157.315) (width 0.25) (layer "F.Cu") (net 32))
   (segment (start 184.296101 153.934452) (end 185.917548 153.934452) (width 0.25) (layer "F.Cu") (net 32))
+  (segment (start 234.28 158.938998) (end 234.28 157.989) (width 0.25) (layer "F.Cu") (net 32))
   (segment (start 237.162 157.989) (end 236.071 157.989) (width 0.25) (layer "F.Cu") (net 32))
   (segment (start 229.414 144.764941) (end 228.357059 143.708) (width 0.25) (layer "F.Cu") (net 32))
@@
   (via (at 199.7769 130.9687) (size 0.8) (drill 0.4) (layers "F.Cu" "B.Cu") (net 32))
   (via (at 223.52 154) (size 0.8) (drill 0.4) (layers "F.Cu" "B.Cu") (net 32))
+  (via (at 234.188 160.528) (size 0.8) (drill 0.4) (layers "F.Cu" "B.Cu") (net 32))
   (via (at 233.5555 148.7685) (size 0.8) (drill 0.4) (layers "F.Cu" "B.Cu") (net 32))
   (via (at 236.071 154.508) (size 0.8) (drill 0.4) (layers "F.Cu" "B.Cu") (net 32))
@@
   (segment (start 221.065511 140.8745) (end 221.038 140.902011) (width 0.25) (layer "B.Cu") (net 32))
   (segment (start 204.034079 145.027984) (end 204.034079 148.163523) (width 0.25) (layer "B.Cu") (net 32))
+  (segment (start 222.2125 154.1405) (end 222.504 154.432) (width 0.25) (layer "B.Cu") (net 32))
   (segment (start 221.224011 140.716) (end 222.221805 140.716) (width 0.25) (layer "B.Cu") (net 32))
   (segment (start 204.034079 145.027984) (end 204.034079 141.913921) (width 0.25) (layer "B.Cu") (net 32))
@@
   (segment (start 234.039 152.476) (end 225.552 152.476) (width 0.25) (layer "B.Cu") (net 32))
   (segment (start 192.241 150.160305) (end 191.816305 150.585) (width 0.25) (layer "B.Cu") (net 32))
+  (segment (start 222.2125 144.581408) (end 222.2125 154.1405) (width 0.25) (layer "B.Cu") (net 32))
+  (segment (start 222.504 154.432) (end 228.6 160.528) (width 0.25) (layer "B.Cu") (net 32))
   (segment (start 204.034079 141.913921) (end 204.724 141.224) (width 0.25) (layer "B.Cu") (net 32))
   (segment (start 222.580378 138.234) (end 213.418 138.234) (width 0.25) (layer "B.Cu") (net 32))
@@
   (segment (start 223.012 137.802378) (end 222.580378 138.234) (width 0.25) (layer "B.Cu") (net 32))
   (segment (start 219.972953 146.820953) (end 220.123 146.670906) (width 0.25) (layer "B.Cu") (net 32))
+  (segment (start 228.6 160.528) (end 234.188 160.528) (width 0.25) (layer "B.Cu") (net 32))
   (segment (start 222.221805 140.716) (end 222.721 141.215195) (width 0.25) (layer "B.Cu") (net 32))
   (segment (start 194.056 148.336) (end 192.241 150.151) (width 0.25) (layer "B.Cu") (net 32))
   (segment (start 236.579 154) (end 236.071 154.508) (width 0.25) (layer "B.Cu") (net 32))
   (segment (start 197.371352 137.656629) (end 197.316473 137.60175) (width 0.25) (layer "F.Cu") (net 33))
-  (segment (start 205.960892 144.257929) (end 204.200963 142.498) (width 0.25) (layer "F.Cu") (net 33))
+  (segment (start 204.200963 142.498) (end 206.482963 144.78) (width 0.25) (layer "F.Cu") (net 33))
   (segment (start 201.887 142.498) (end 201.025374 141.636374) (width 0.25) (layer "F.Cu") (net 33))
   (segment (start 197.223741 141.636374) (end 196.533741 142.326374) (width 0.25) (layer "F.Cu") (net 33))
-  (segment (start 204.200963 142.498) (end 201.887 142.498) (width 0.25) (layer "F.Cu") (net 33))
-  (segment (start 207.202706 144.257929) (end 205.960892 144.257929) (width 0.25) (layer "F.Cu") (net 33))
+  (segment (start 206.482963 144.78) (end 207.202706 144.78) (width 0.25) (layer "F.Cu") (net 33))
+  (segment (start 201.887 142.498) (end 204.200963 142.498) (width 0.25) (layer "F.Cu") (net 33))
   (segment (start 196.533741 140.209556) (end 197.371352 139.371945) (width 0.25) (layer "F.Cu") (net 33))
   (segment (start 197.371352 139.371945) (end 197.371352 137.656629) (width 0.25) (layer "F.Cu") (net 33))

Commit message: new fixes
Parts:
- removed C21: C 1uF/16V (10%), Capacitor_SMD:C_0603_1608Metric
- removed C22: 4.7uF, Capacitor_SMD:C_0603_1608Metric
- removed C23: 0.1 uF, Capacitor_SMD:C_0603_1608Metric
- removed D7, D8, D9: LESD5D5.0CT1G, LESD5D5.0CT1G:TVS_LESD5D5.0CT1G
- removed Q1, Q2: BC818, Package_TO_SOT_SMD:SOT-23
- removed R17: R 22.1k (1%), Resistor_SMD:R_0603_1608Metric
- removed R22: R 47.5k (1%), Resistor_SMD:R_0603_1608Metric
- removed R23: 1K(1%), Resistor_SMD:R_0603_1608Metric
- removed R24, R25, R26: R 10k (1%), Resistor_SMD:R_0603_1608Metric
- removed U3: CP2102N-A02-GQFN28R, CP2102N-A02-GQFN28R:IC_CP2102N-A02-GQFN28R
- added C4: 0.1uF, Capacitor_SMD:C_0603_1608Metric, F.Cu at (180.3, 155.4)
- added C5: 1uF, Capacitor_SMD:C_0603_1608Metric, F.Cu at (189.0, 128.0)
- added D12: TPD4E1B06DCKR, TPD4E1B06DCKR:TVS_TPD4E1B06DCKR, F.Cu at (206.3, 145.9)
- added R10: R 2.2k, Capacitor_SMD:C_0402_1005Metric, F.Cu at (252.0, 128.0)
- added R11: R 2.2k, Capacitor_SMD:C_0402_1005Metric, F.Cu at (252.0, 133.1)
- added R12: R 2.2k, Capacitor_SMD:C_0402_1005Metric, F.Cu at (252.4, 139.7)
- added R13: R 2.2k, Capacitor_SMD:C_0402_1005Metric, F.Cu at (252.5, 144.3)
- added R14: R 2.2k, Capacitor_SMD:C_0402_1005Metric, F.Cu at (252.5, 149.4)
- added R15: R 2.2k, Capacitor_SMD:C_0402_1005Metric, F.Cu at (252.0, 129.0)
- added R16: R 2.2k, Capacitor_SMD:C_0402_1005Metric, F.Cu at (252.0, 134.1)
- added R18: R 2.2k, Capacitor_SMD:C_0402_1005Metric, F.Cu at (252.4, 140.7)
- added R19: R 2.2k, Capacitor_SMD:C_0402_1005Metric, F.Cu at (252.5, 145.3)
- added R20: R 2.2k, Capacitor_SMD:C_0402_1005Metric, F.Cu at (252.5, 150.4)
- added R21: R 2.2k, Capacitor_SMD:C_0402_1005Metric, F.Cu at (252.0, 130.0)
- added R29: R 2.2k, Capacitor_SMD:C_0402_1005Metric, F.Cu at (252.0, 135.1)
- added R7: R 2.2k, Capacitor_SMD:C_0402_1005Metric, F.Cu at (252.5, 138.7)
- added R8: R 2.2k, Capacitor_SMD:C_0402_1005Metric, F.Cu at (252.5, 143.3)
- added R9: R 2.2k, Capacitor_SMD:C_0402_1005Metric, F.Cu at (252.5, 148.3)
- added S1: TS-1187A-B-A-B, TS-1187A-B-A-B:SW_TS-1187A-B-A-B, F.Cu at (183.9, 128.5)
- added S2: TS-1187A-B-A-B, TS-1187A-B-A-B:SW_TS-1187A-B-A-B, F.Cu at (184.9, 160.0)
- C19: footprint Capacitor_SMD:C_0805_2012Metric -> Capacitor_SMD:C_1206_3216Metric
- D11: value BLUE LED -> EMERALD LED
- R1, R2, R3, R4, R5: value CAT10-222J4LF -> R 2.2k; footprint CAT10-222J4LF:RESCAV50P200X100X55-8N -> Capacitor_SMD:C_0402_1005Metric
- R27: value 5.1 -> 100
- moved C56 25.6 mm to (243.8, 128.0)
- moved R28 25.6 mm to (243.8, 129.5)
- moved R4 21.8 mm to (252.0, 127.0), turned to 180 degrees
- moved R2 8.76 mm to (252.5, 142.2), turned to 180 degrees
- moved R5 3.81 mm to (252.0, 132.1), turned to 180 degrees
- moved R3 3.30 mm to (252.5, 147.3), turned to 180 degrees
- moved C38 1.61 mm to (237.7, 127.0)
- moved C20 1.61 mm to (237.7, 129.0)
- moved R1 1.49 mm to (252.5, 137.7), turned to 180 degrees
- moved C19 0.81 mm to (233.7, 129.5)
Connections:
- net /EN renamed Net-(U12-EN)
- J1 pad 2: /USB Port/USBtoUART/DN -> /DN
- J1 pad 3: /USB Port/USBtoUART/DP -> /DP
- R1 pad 1: /IN3P -> /3P
- R1 pad 2: /IN3N -> /IN3P
- R2 pad 1: /IN1P -> /5P
- R2 pad 2: /IN1N -> /IN5P
- R3 pad 1: /IN5P -> /7P
- R3 pad 2: /IN5N -> /IN7P
- R4 pad 1: /IN7P -> /SRB1
- R4 pad 2: /IN7N -> /INSRB1
- R5 pad 1: /INSRB1 -> /1P
- R5 pad 2: /INSRB2 -> /IN1P
- U10 pad 1: GNDA -> /INSRB1
- U10 pad 2: GNDA -> /INSRB1
- U10 pad 3: GNDA -> /INSRB1
- U10 pad 4: GNDA -> /INSRB1
- U11 pad 1: GNDA -> /INSRB1
- U11 pad 2: GNDA -> /INSRB1
- U11 pad 3: GNDA -> /INSRB1
- U11 pad 4: GNDA -> /INSRB1
- U12 pad 23: unconnected-(U12-GPIO19/U1RTS/ADC2_CH8/CLK_OUT2/USB_D--Pad23) -> /DN
- U12 pad 24: unconnected-(U12-GPIO20/U1CTS/ADC2_CH9/CLK_OUT1/USB_D+-Pad24) -> /DP
- U12 pad 4: /GPIO0 -> Net-(U12-GPIO0/BOOT)
- U7 pad 1: GNDA -> /INSRB1
- U7 pad 2: GNDA -> /INSRB1
- U7 pad 3: GNDA -> /INSRB1
- U7 pad 4: GNDA -> /INSRB1
- U8 pad 1: GNDA -> /INSRB1
- U8 pad 2: GNDA -> /INSRB1
- U8 pad 3: GNDA -> /INSRB1
- U8 pad 4: GNDA -> /INSRB1
- U9 pad 1: GNDA -> /INSRB1
- U9 pad 2: GNDA -> /INSRB1
- U9 pad 3: GNDA -> /INSRB1
- U9 pad 4: GNDA -> /INSRB1
Routing:
- net GNDA: track 194.8 -> 129.1 mm, vias 17 -> 12
- net /INSRB1: track 22.0 -> 64.1 mm, vias 2 -> 6
- net /USB Port/USBtoUART/DP: track 39.9 -> 0.00 mm, vias 2 -> 0
- net /USB Port/USBtoUART/DN: track 38.0 -> 0.00 mm, vias 2 -> 0
- net /GPIO0: track 32.7 -> 0.00 mm, vias 2 -> 0
- net /DP: track 0.00 -> 31.4 mm
- net /DN: track 0.00 -> 29.7 mm
- net GND: track 253.2 -> 225.8 mm, vias 16 -> 13
- net Net-(U12-GPIO0/BOOT): track 0.00 -> 21.6 mm, vias 0 -> 2
- net /BIAS_DRV: track 28.0 -> 9.92 mm, vias 2 -> 0
- net /U0RXD: track 16.5 -> 0.00 mm, vias 2 -> 0
- net /U0TXD: track 15.6 -> 0.00 mm
- net /USB Port/USBtoUART/DTR: track 14.0 -> 0.00 mm, vias 3 -> 0
- net VBUS: track 35.7 -> 22.2 mm, vias 0 -> 2
- net /USB Port/USBtoUART/RTS: track 13.4 -> 0.00 mm
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Other:
- board text added: "Monolith BCI 0.2"
- board text removed: "Monolith BCI"

Commit message: wahoo
Parts:
- added REF**: OSHW-Logo2_14.6x12mm_SilkScreen, Symbol:OSHW-Logo2_14.6x12mm_SilkScreen, F.Cu at (210.1, 156.2)
Routing:
- net /DN: track 29.7 -> 31.0 mm

Commit message: ready to fab?
Parts:
- added G***: LOGO, LOGO, B.Cu at (237.2, 142.7)
- added G***: LOGO, LOGO, B.Cu at (199.4, 142.7)
- moved REF** 8.18 mm to (202.7, 152.7)
Other:
- board text added: "+3V3"
- board text added: "BOOT"
- board text added: "CS"
- board text added: "DIN"
- board text added: "DOUT"
- board text added: "GND"
- board text added: "Monolith BCI - 0.2"
- board text added: "RESET"
- board text added: "SCLK"
- board text added: "~{DRDY}"
- board text added: "~{RESET}"
- board text removed: "Monolith BCI 0.2"

Commit message: fix pin headers
Parts:
- removed the REF** at (202.7, 152.7)
- added REF**: ESD-Logo_6.6x6mm_SilkScreen, Symbol:ESD-Logo_6.6x6mm_SilkScreen, F.Cu at (247.9, 157.7)
- added REF**: OSHW-Symbol_8.9x8mm_SilkScreen, Symbol:OSHW-Symbol_8.9x8mm_SilkScreen, F.Cu at (205.0, 153.9)
- J2, J3: footprint Connector_PinSocket_2.54mm:PinSocket_1x11_P2.54mm_Vertical -> Connector_PinHeader_2.54mm:PinHeader_1x11_P2.54mm_Vertical
- J4, J5: footprint Connector_PinSocket_2.54mm:PinSocket_1x02_P2.54mm_Vertical -> Connector_PinHeader_2.54mm:PinHeader_1x02_P2.54mm_Vertical
- J7: footprint Connector_PinHeader_2.54mm:PinHeader_1x08_P2.54mm_Vertical -> Connector_PinSocket_2.54mm:PinSocket_1x08_P2.54mm_Vertical

Commit message: change text
Other:
- board text added: "Monolith BCI 0.2"
- board text removed: "Monolith BCI - 0.2"
