File: Monolith.kicad_pcb (KiCad board)
At the start: 2 copper layers, 89.9 x 42.7 mm, 91 parts, among them J1 USB_B_Micro, J2 Conn_01x11, J3 Conn_01x11, J4 Conn_01x02, J5 Conn_01x02, J7 Conn_01x08, U1 ADS1299IPAGR, U12 ESP32-S3-MINI-1, U2 AMS1117-3.3, U4 LM2664M6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

Commit message: fix reset button
Parts:
- removed C5: 1uF, Capacitor_SMD:C_0603_1608Metric
- removed REF**: ESD-Logo_6.6x6mm_SilkScreen, Symbol:ESD-Logo_6.6x6mm_SilkScreen
- removed REF**: OSHW-Symbol_8.9x8mm_SilkScreen, Symbol:OSHW-Symbol_8.9x8mm_SilkScreen
- added C6: 0.1uF, Capacitor_SMD:C_0603_1608Metric, F.Cu at (189.0, 128.0)
Connections:
- S1 pad A: Net-(C5-Pad1) -> GND
- S1 pad B: Net-(C5-Pad1) -> GND
Routing:
- net Net-(C5-Pad1): track 8.30 -> 0.00 mm
- net GND: track 225.8 -> 221.8 mm
- net Net-(U12-EN): track 20.7 -> 23.1 mm
